Commit message: added non functional mecanum drive

File: summit_xl_description/urdf/bases/summit_xl_base.gazebo.xacro (robot description, xacro)
@@ -16,7 +16,5 @@
 	<xacro:macro name="skid_steering" params="prefix publish_tf">
     <gazebo>
-      <!-- <plugin name="skid_steer_drive_controller" filename="libgazebo_ros_diff_drive.so"> -->
 	  <plugin filename="gz-sim-diff-drive-system" name="gz::sim::systems::DiffDrive">
-			<!--<robotNamespace>/summit_xl</robotNamespace>-->
 		    <odom_publish_frequency>50.0</odom_publish_frequency>
 		    <left_joint>${prefix}front_left_wheel_joint</left_joint>
@@ -24,15 +22,11 @@
 		    <left_joint>${prefix}back_left_wheel_joint</left_joint>
 		    <right_joint>${prefix}back_right_wheel_joint</right_joint>
-		    <!-- wheelSeparation>0.566</wheelSeparation --> <!-- real parameter value -->
+		    <!-- wheel_separation>0.566</wheel_separation --> <!-- real parameter value -->
 		    <wheel_separation>0.462</wheel_separation> <!-- works a bit better in Gazebo -->
 		    <wheel_radius>0.11</wheel_radius>
 		    <child_frame_id>${prefix}base_footprint</child_frame_id>
-		    <!-- <torque>50</torque> -->
-			<ros>
-				<remapping>cmd_vel:=/robotnik_base_control/cmd_vel</remapping>
-         		<remapping>odom:=/robotnik_base_control/odom</remapping>
-			</ros>
+			<topic>/robotnik_base_control/cmd_vel</topic>
+         	<odom_topic>/robotnik_base_control/odom</odom_topic>
 		    <frame_id>${prefix}odom</frame_id>
-		    <broadcastTF>${publish_tf}</broadcastTF>
       </plugin>
     </gazebo>
@@ -40,46 +34,13 @@
   <xacro:macro name="omni_steering" params="namespace publish_tf">
 		<gazebo>
-	    <!-- <plugin name="omni_steering" filename="libgazebo_ros_planar_move.so">
-	      <commandTopic>robotnik_base_control/cmd_vel</commandTopic>
-	      <odometryTopic>robotnik_base_control/odom</odometryTopic>
-	      <odometryFrame>${prefix}odom</odometryFrame>
-	      <odometryRate>50.0</odometryRate>
-	      <robotBaseFrame>${prefix}base_footprint</robotBaseFrame>
-	      <publishTF>${publish_tf}</publishTF>
-		  <enableYAxis>true</enableYAxis>
-	    </plugin> -->
-		<plugin name='planar_move' filename='libgazebo_ros_planar_move.so'>
-        <ros>
-          <namespace>${namespace}</namespace>
-		  <remapping>/tf:=tf</remapping>
-          <!-- <remapping>cmd_vel:=robotnik_base_control/cmd_vel</remapping>
-          <remapping>odom:=robotnik_base_control/odom</remapping> -->
-        </ros>
-        <update_rate>100</update_rate>
-        <publish_rate>100</publish_rate>
-        <publish_odom>true</publish_odom>
-        <publish_odom_tf>${publish_tf}</publish_odom_tf>
-        <odometry_frame>odom</odometry_frame> <!-- TOF: was ${namespace}/odom -->
-        <robot_base_frame>base_footprint</robot_base_frame> <!-- TOF: was ${namespace}/base_footprint-->
+		<plugin name='gz-sim-mecanum-drive-system' filename="gz::sim::systems::MecanumDrive">
+		<topic>/robotnik_base_control/cmd_vel</topic>
+        <odom_topic>/robotnik_base_control/odom</odom_topic>
+		<publish_odom_tf>${publish_tf}</publish_odom_tf>
+        <frame_id>odom</frame_id> <!-- TOF: was ${namespace}/odom -->
+        <child_frame_id>base_footprint</child_frame_id> <!-- TOF: was ${namespace}/base_footprint-->
       </plugin>
 	  </gazebo>
   </xacro:macro>
-  	<xacro:macro name="skid_steering" params="prefix publish_tf">
-		<gazebo>
-			<plugin name="skid_steering" filename="libgazebo_ros_planar_move.so">
-			<ros>
-				<remapping>cmd_vel:=/robotnik_base_control/cmd_vel</remapping>
-         		<remapping>odom:=/robotnik_base_control/odom</remapping>
-			<!-- <commandTopic>robotnik_base_control/cmd_vel</commandTopic> -->
-			<!-- <odometryTopic>robotnik_base_control/odom</odometryTopic> -->
-			</ros>
-			<odometryFrame>${prefix}odom</odometryFrame>
-			<odometryRate>50.0</odometryRate>
-			<robotBaseFrame>${prefix}base_footprint</robotBaseFrame>
-			<publishTF>${publish_tf}</publishTF>
-			<enableYAxis>false</enableYAxis>
-			</plugin>
-		</gazebo>
-  	</xacro:macro>
   <xacro:macro name="ros_force_based_move" params="publish_tf prefix">
 	  <gazebo>

Commit message: update

File: summit_xl_description/urdf/bases/summit_xl_base.gazebo.xacro (robot description, xacro)
@@ -32,12 +32,21 @@
     </gazebo>
   </xacro:macro>
-  <xacro:macro name="omni_steering" params="namespace publish_tf">
+  <xacro:macro name="omni_steering" params="prefix publish_tf">
 		<gazebo>
-		<plugin name='ignition-gazebo-mecanum-drive-system' filename="ignition::gazebo::systems::MecanumDrive">
-		<topic>/robotnik_base_control/cmd_vel</topic>
-        <odom_topic>/robotnik_base_control/odom</odom_topic>
-		<publish_odom_tf>${publish_tf}</publish_odom_tf>
-        <frame_id>odom</frame_id> <!-- TOF: was ${namespace}/odom -->
-        <child_frame_id>base_footprint</child_frame_id> <!-- TOF: was ${namespace}/base_footprint-->
+		<plugin filename='ignition-gazebo-mecanum-drive-system' name="ignition::gazebo::systems::MecanumDrive">
+			<odom_publish_frequency>50.0</odom_publish_frequency>
+			<front_left_joint>${prefix}front_left_wheel_joint</front_left_joint>
+			<front_right_joint>${prefix}front_right_wheel_joint</front_right_joint>
+			<back_left_joint>${prefix}back_left_wheel_joint</back_left_joint>
+			<back_right_joint>${prefix}back_right_wheel_joint</back_right_joint>
+			<!-- https://www.roscomponents.com/en/mobile-robots/rb-steel -->
+			<wheel_separation>0.535</wheel_separation>
+			<wheelbase>0.43</wheelbase>
+			<wheel_radius>0.127</wheel_radius>
+			<topic>/robotnik_base_control/cmd_vel</topic>
+			<odom_topic>/robotnik_base_control/odom</odom_topic>
+			<tf_topic>${publish_tf}</tf_topic>
+			<frame_id>${prefix}odom</frame_id>
+			<child_frame_id>${prefix}base_footprint</child_frame_id>
       </plugin>
 	  </gazebo>

File: summit_xl_description/urdf/ros2_control.urdf.xacro (robot description, xacro)
@@ -4,5 +4,5 @@
       <gazebo>
         <!-- <plugin name="ros_control" filename="libgazebo_ros2_control.so"> -->
-        <plugin filename="libgz_ros2_control-system.so" name="gz_ros2_control::GazeboSimROS2ControlPlugin">
+        <plugin filename="ign_ros2_control-system" name="ign_ros2_control::IgnitionROS2ControlPlugin">
           <ros>
             <namespace>$(arg robot_id)</namespace>
@@ -14,5 +14,5 @@
         <hardware>
           <!-- <plugin>gazebo_ros2_control/GazeboSystem</plugin> -->
-          <plugin>gz_ros2_control/GazeboSimSystem</plugin>
+          <plugin>ign_ros2_control/IgnitionSystem</plugin>
         </hardware>
         <joint name="front_left_wheel_joint">

File: summit_xl_description/urdf/sensors/hokuyo_ust20lx_no_frame_prefix.urdf.xacro (robot description, xacro)
@@ -36,9 +36,9 @@
   <xacro:macro name="sensor_hokuyo_ust20_gazebo_no_frame_prefix">
     <gazebo reference="${prefix}_link">
-			<sensor type="ray" name="${prefix}_sensor">
+			<sensor type="gpu_lidar" name="${prefix}_sensor">
 				<pose>0 0 0 0 0 0</pose>
 				<topic>lidar</topic>
 				<update_rate>40</update_rate>
-				<ray>
+				<lidar>
 					<scan>
 						<horizontal>
@@ -59,6 +59,6 @@
 						<stddev>0.01</stddev>
 					</noise>
-				</ray>
-        <always_on>1</always_on>
+				</lidar>
+        <always_on>true</always_on>
         <visualize>true</visualize>
 				<!-- <plugin name="${prefix}" filename="libgazebo_ros_ray_sensor.so"> -->
@@ -71,5 +71,6 @@
           </ros>
           <output_type>sensor_msgs/LaserScan</output_type>
-          <frame_name>${prefix}_link</frame_name>
+          <!-- <frame_name>${prefix}_link</frame_name> -->
+          <gz_frame_id>${prefix}_link</gz_frame_id>
 				</plugin>
 			</sensor>
